File: hardware/micropad/micropad.sch (KiCad schematic (older format))
At the start: 31 parts, among them J1 SWD Debug, J2 USB_C_Receptacle_USB2.0, SW1 SW_SPST, SW2 SW_SPST, SW3 SW_SPST, U1 LD1117S33TR_SOT223, U2 STM32F042K6Ux, U3 APA102

Commit message: Change PCB mounting holes to M3
Parts:
- H1, H2, H3, H4: footprint Mounting_Holes:MountingHole_2.2mm_M2_ISO7380_Pad -> Mounting_Holes:MountingHole_3.2mm_M3_ISO7380_Pad
Changed lines of the file:
@@
 F 0 "H1" H 2500 5096 50  0000 L CNN
 F 1 "MountingHole" H 2500 5005 50  0000 L CNN
-F 2 "Mounting_Holes:MountingHole_2.2mm_M2_ISO7380_Pad" H 2400 5050 50  0001 C CNN
+F 2 "Mounting_Holes:MountingHole_3.2mm_M3_ISO7380_Pad" H 2400 5050 50  0001 C CNN
 F 3 "~" H 2400 5050 50  0001 C CNN
 	1    2400 5050
@@
 F 0 "H2" H 2500 5346 50  0000 L CNN
 F 1 "MountingHole" H 2500 5255 50  0000 L CNN
-F 2 "Mounting_Holes:MountingHole_2.2mm_M2_ISO7380_Pad" H 2400 5300 50  0001 C CNN
+F 2 "Mounting_Holes:MountingHole_3.2mm_M3_ISO7380_Pad" H 2400 5300 50  0001 C CNN
 F 3 "~" H 2400 5300 50  0001 C CNN
 	1    2400 5300
@@
 F 0 "H3" H 2500 5596 50  0000 L CNN
 F 1 "MountingHole" H 2500 5505 50  0000 L CNN
-F 2 "Mounting_Holes:MountingHole_2.2mm_M2_ISO7380_Pad" H 2400 5550 50  0001 C CNN
+F 2 "Mounting_Holes:MountingHole_3.2mm_M3_ISO7380_Pad" H 2400 5550 50  0001 C CNN
 F 3 "~" H 2400 5550 50  0001 C CNN
 	1    2400 5550
@@
 F 0 "H4" H 2500 5846 50  0000 L CNN
 F 1 "MountingHole" H 2500 5755 50  0000 L CNN
-F 2 "Mounting_Holes:MountingHole_2.2mm_M2_ISO7380_Pad" H 2400 5800 50  0001 C CNN
+F 2 "Mounting_Holes:MountingHole_3.2mm_M3_ISO7380_Pad" H 2400 5800 50  0001 C CNN
 F 3 "~" H 2400 5800 50  0001 C CNN
 	1    2400 5800
